Commit message: Added camera.xacro to description folder

File: ppp_bot/description/ignition_control.xacro (robot description, xacro)
@@ -1,4 +1,4 @@
 <?xml version="1.0"?>
-<robot xmlns:xacro="http://www.ros.org/wiki/xacro" name="robot">
+<robot xmlns:xacro="http://www.ros.org/wiki/xacro">
     <gazebo>
         <plugin

File: ppp_bot/description/lidar.xacro (robot description, xacro)
@@ -23,30 +23,30 @@
     </link>
     <gazebo reference="lidar_frame">
-        <sensor name='gpu_lidar' type='gpu_lidar'>
-          <topic>lidar</topic>
-          <update_rate>10</update_rate>
-          <lidar>
-            <scan>
-              <horizontal>
-                <samples>640</samples>
-                <resolution>1</resolution>
-                <min_angle>-1.396263</min_angle>
-                <max_angle>1.396263</max_angle>
-              </horizontal>
-              <vertical>
-                <samples>16</samples>
-                <resolution>1</resolution>
-                <min_angle>-0.261799</min_angle>
-                <max_angle>0.261799</max_angle>
-              </vertical>
-            </scan>
-            <range>
-              <min>0.08</min>
-              <max>10.0</max>
-              <resolution>0.01</resolution>
-            </range>
-          </lidar>
-          <visualize>true</visualize>
-        </sensor>
+      <sensor name='gpu_lidar' type='gpu_lidar'>
+        <topic>lidar</topic>
+        <update_rate>10</update_rate>
+        <lidar>
+          <scan>
+            <horizontal>
+              <samples>640</samples>
+              <resolution>1</resolution>
+              <min_angle>-1.396263</min_angle>
+              <max_angle>1.396263</max_angle>
+            </horizontal>
+            <vertical>
+              <samples>1</samples>
+              <resolution>1</resolution>
+              <min_angle>0.0</min_angle>
+              <max_angle>0.0</max_angle>
+            </vertical>
+          </scan>
+          <range>
+            <min>0.08</min>
+            <max>10.0</max>
+            <resolution>0.01</resolution>
+          </range>
+        </lidar>
+        <visualize>true</visualize>
+      </sensor>
     </gazebo>
 </robot>

File: ppp_bot/description/materials.xacro (robot description, xacro)
@@ -1,4 +1,4 @@
 <?xml version="1.0"?>
-<robot xmlns:xacro="http://www.ros.org/wiki/xacro" name="robot">
+<robot xmlns:xacro="http://www.ros.org/wiki/xacro">
     <material name="white">
         <color rgba="1 1 1 1" />

File: ppp_bot/description/robot.urdf (robot description, URDF)
Before this commit: robot robot, 6 links, 5 joints
Links:
- added link camera_link; visual box size=0.010 0.03 0.03
- added link camera_link_optical
Joints:
- added joint camera_joint: type fixed, parent chassis, child camera_link, origin xyz=0.305 0 0.08 rpy=0 0 0
- added joint camera_optical_joint: type fixed, parent camera_link, child camera_link_optical, origin xyz=0 0 0 rpy=-1.5707963267948966 0 -1.5707963267948966

File: ppp_bot/description/robot.urdf.xacro (robot description, xacro)
@@ -3,3 +3,4 @@
     <xacro:include filename="robot_core.xacro" />
     <xacro:include filename="lidar.xacro" />
+    <xacro:include filename="camera.xacro" />
 </robot>
