Commit message: Added depth camera

File: ppp_bot/description/depth_camera.xacro (robot description, xacro)
@@ -1,10 +1,10 @@
 <?xml version="1.0"?>
-<robot xmlns:xacro="http://www.ros.org/wiki/xacro">
-    <joint name="camera_joint" type="fixed">
+<robot xmlns:xacro="http://www.ros.org/wiki/xacro" >
+    <joint name="depth_camera_joint" type="fixed">
         <parent link="chassis"/>
-        <child link="camera_link"/>
+        <child link="depth_camera_link"/>
         <origin xyz="0.305 0 0.08" rpy="0 0 0"/>
     </joint>
-    <link name="camera_link">
+    <link name="depth_camera_link">
         <visual>
             <geometry>
@@ -13,15 +13,13 @@
             <material name="red"/>
         </visual>
-    </link>            <plugin name="camera_controller" filename="libgazebo_ros_camera.so">
-                <frame_name>camera_link_optical</frame_name>
-            </plugin>
-    <joint name="camera_optical_joint" type="fixed">
-        <parent link="camera_link"/>
-        <child link="camera_link_optical"/>
+    </link>
+    <joint name="depth_camera_optical_joint" type="fixed">
+        <parent link="depth_camera_link"/>
+        <child link="depth_camera_link_optical"/>
         <origin xyz="0 0 0" rpy="${-pi/2} 0 ${-pi/2}"/>
     </joint>
-    <link name="camera_link_optical"></link>
-    <gazebo reference="camera_link">
-        <sensor name="camera" type="camera">
+    <link name="depth_camera_link_optical"></link>
+    <gazebo reference="depth_camera_link">
+        <sensor name="depth_camera" type="depth">
             <pose> 0 0 0 0 0 0 </pose>
             <visualize>true</visualize>
@@ -30,5 +28,5 @@
                 <horizontal_fov>1.089</horizontal_fov>
                 <image>
-                    <format>R8G8B8</format>
+                    <format>B8G8R8</format>
                     <width>640</width>
                     <height>480</height>

File: ppp_bot/description/robot.urdf (robot description, URDF)
Before this commit: robot robot, 8 links, 7 joints
Links:
- added link depth_camera_link; visual box size=0.010 0.03 0.03
- added link depth_camera_link_optical
Joints:
- added joint depth_camera_joint: type fixed, parent chassis, child depth_camera_link, origin xyz=0.305 0 0.08 rpy=0 0 0
- added joint depth_camera_optical_joint: type fixed, parent depth_camera_link, child depth_camera_link_optical, origin xyz=0 0 0 rpy=-1.5707963267948966 0 -1.5707963267948966

File: ppp_bot/description/robot.urdf.xacro (robot description, xacro)
@@ -4,3 +4,4 @@
     <xacro:include filename="lidar.xacro" />
     <xacro:include filename="camera.xacro" />
+    <xacro:include filename="depth_camera.xacro" />
 </robot>
