Commit message: Added cones world and world_name launch configuration to launch_sim.launch.py

File: ppp_bot/description/lidar.xacro (robot description, xacro)
@@ -24,5 +24,5 @@
     <gazebo reference="lidar_frame">
       <sensor name='gpu_lidar' type='gpu_lidar'>
-        <topic>lidar</topic>
+        <topic>scan</topic>
         <update_rate>10</update_rate>
         <lidar>

File: ppp_bot/description/robot.urdf (robot description, URDF)
Before this commit: robot robot, 10 links, 9 joints
Links:
- added link base_footprint
Joints:
- added joint base_footprint_joint: type fixed, parent base_link, child base_footprint, origin xyz=0 0 0 rpy=0 0 0

File: ppp_bot/description/robot_core.xacro (robot description, xacro)
@@ -5,4 +5,12 @@
     <!-- BASE LINK -->
     <link name="base_link">
+    </link>
+    <!-- BASE_FOOTPRINT LINK -->
+    <joint name="base_footprint_joint" type="fixed">
+        <parent link="base_link"/>
+        <child link="base_footprint"/>
+        <origin xyz="0 0 0" rpy="0 0 0"/>
+    </joint>
+    <link name="base_footprint">
     </link>
     <!-- CHASSIS LINK -->

Commit message: Added rviz and smoother robot control

File: ppp_bot/description/lidar.xacro (robot description, xacro)
@@ -43,5 +43,5 @@
           <range>
             <min>0.08</min>
-            <max>10.0</max>
+            <max>20.0</max>
             <resolution>0.01</resolution>
           </range>

File: ppp_bot/description/robot.urdf (robot description, URDF)
Before this commit: robot robot, 11 links, 10 joints
Links:
- removed link depth_camera_link
- removed link depth_camera_link_optical
Joints:
- removed joint depth_camera_joint
- removed joint depth_camera_optical_joint

File: ppp_bot/description/robot.urdf.xacro (robot description, xacro)
@@ -4,4 +4,4 @@
     <xacro:include filename="lidar.xacro" />
     <xacro:include filename="camera.xacro" />
-    <xacro:include filename="depth_camera.xacro" />
+    <!-- <xacro:include filename="depth_camera.xacro" /> -->
 </robot>
